Commit message: 2021-8-10 clear the workspace

File: src/armbot_description/urdf/husky.urdf (robot description, URDF)
Before this commit: robot husky, 15 links, 14 joints
Links:
- removed link ouster_laser_link
- added link base_scan; visual mesh filename=package://armbot_description/meshes/laser_link.STL
Joints:
- joint ouster_laser_extension: child ouster_laser_link -> base_scan
